File: power.kicad_sch (KiCad schematic)
At the start: 26 parts, among them J1 USB_C_Receptacle_USB2.0_14P, J2 Conn_01x02, Q1 NMOS, Q2 NMOS, U1 TPS63802DLAR, U2 TP4056-42-ESOP8, U3 DW01A

Commit message: finalized the schematic design
Parts:
- added D3: ESD5Zxx, Diode_SMD:D_SOD-523, symbol Diode:ESD5Zxx
- C1, C2, C3, C5: footprint (none) -> Capacitor_SMD:C_0805_2012Metric
- C4: footprint (none) -> Capacitor_SMD:C_0603_1608Metric
- D1, D2: footprint (none) -> LED_SMD:LED_0603_1608Metric
- J1: footprint (none) -> Connector_USB:USB_C_Receptacle_GCT_USB4085
- L1: footprint (none) -> ul_XFL4015-471MEC:IND_XFL4015_COC-M
- Q1, Q2: footprint (none) -> Package_TO_SOT_SMD:SOT-23
- R1, R10, R11, R2, R3, R4, R5, R6, R7, R8, R9: footprint (none) -> Resistor_SMD:R_0603_1608Metric
Connections:
- net GND: now also D3.1 (K)
- net at C3.1, D1.2 (A), D2.2 (A)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: now also D3.2 (A)
- net BATT+: now reaches C1.1, C4.2, C5.2, J2.1 (Pin_1), R11.2, U1.1 (EN), U1.10 (VIN), U2.5 (BAT)
- net D+: no longer names the net of J1.A6 (D+)
- net D+: no longer J1.B6 (D+)
- net D-: no longer names the net of J1.A7 (D-)
- net D-: no longer J1.B7 (D-)
- no-connect marks 0 -> 4
Other:
- moved on the sheet: C3
