File: sensor_node_kicad.kicad_sch (KiCad schematic)
At the start: 0 parts

Commit message: progressed in the processing unit, BME280 still needs proper implementation
Other:
- added sheet Processing (processing.kicad_sch)
Changed lines of the file:
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@@
 	(generator_version "9.0")
 	(paper "A4")
+	(wire
+		(pts
+			(xy 121.92 71.12) (xy 146.05 71.12)
+		)
+		(stroke
+			(width 0)
+			(type default)
+		)
+	)
 	(sheet
 		(at 33.02 50.8)
@@
 				)
 			)
+		)
+	)
+	(sheet
+		(at 146.05 49.53)
+		(size 114.3 46.99)
+		(exclude_from_sim no)
+		(in_bom yes)
+		(on_board yes)
+		(dnp no)
+		(fields_autoplaced yes)
+		(stroke
+			(width 0.1524)
+			(type solid)
+		)
+		(fill
+			(color 0 0 0 0.0000)
+		)
+		(property "Sheetname" "Processing"
+			(at 146.05 48.8184 0)
+			(effects
+				(font
+					(size 1.27 1.27)
+				)
+				(justify left bottom)
+			)
+		)
+		(property "Sheetfile" "processing.kicad_sch"
+			(at 146.05 97.1046 0)
+			(effects
+				(font
+					(size 1.27 1.27)
+				)
+				(justify left top)
+			)
+		)
+		(pin "3V3" input
+			(at 146.05 71.12 180)
+			(effects
+				(font
+					(size 1.27 1.27)
+				)
+				(justify left)
+			)
+		)
+		(instances
+			(project "sensor_node_kicad"
+				(path "/f70c476d-7bbd-4b06-90f6-4e1ba7eb4803"
+					(page "3")
+				)
+			)

Commit message: finalized the schematic design
Other:
- sheet Processing renamed Sensor Node Core
- sheet Power ports: added BATT+; removed D+, D-
- sheet Sensor Node Core ports: added BATT+; removed none
Changed lines of the file:
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@@
+		)
+	)
+	(wire
+		(pts
+			(xy 121.92 82.55) (xy 146.05 82.55)
+		)
+		(stroke
+			(width 0)
+			(type default)
 		)
 	)
@@
 			)
 		)
-		(pin "D-" bidirectional
-			(at 83.82 93.98 270)
+		(pin "3V3" output
+			(at 121.92 71.12 0)
 			(effects
 				(font
 					(size 1.27 1.27)
 				)
-				(justify left)
+				(justify right)
 			)
 		)
-		(pin "D+" bidirectional
-			(at 73.66 93.98 270)
-			(effects
-				(font
-					(size 1.27 1.27)
-				)
-				(justify left)
-			)
-		)
-		(pin "3V3" output
-			(at 121.92 71.12 0)
+		(pin "BATT+" output
+			(at 121.92 82.55 0)
 			(effects
 				(font
@@
 			(color 0 0 0 0.0000)
 		)
-		(property "Sheetname" "Processing"
+		(property "Sheetname" "Sensor Node Core"
 			(at 146.05 48.8184 0)
 			(effects
@@
 			(effects
 				(font
+					(size 1.27 1.27)
+				)
+				(justify left)
+			)
+		)
+		(pin "BATT+" input
+			(at 146.05 82.55 180)
+			(effects
+				(font
